Commit message: fixed include and added second camera in the back

File: sensors/d435_camera.urdf.xacro (robot description, xacro)
@@ -1,5 +1,5 @@
 <?xml version="1.0"?>
 <robot xmlns:xacro="http://ros.org/wiki/xacro">
-<xacro:include filename="$(find ur_description)/gazebo/d435_camera_openni.gazebo.urdf.xacro"/>
+<xacro:include filename="$(find ur_description)/sensors/d435_camera_openni.gazebo.urdf.xacro"/>
 <xacro:property name="M_PI" value="3.1415926535897931" />
 <!-- The following values are approximate, and the camera node publishing TF values with actual calibrated camera extrinsic values -->

File: urdf/ur5.xacro (robot description, xacro)
@@ -44,4 +44,15 @@
 		camera_plugin="true">
 		<origin xyz="0.05 0.0 -0.02" rpy="0 -1.57 0.0"/>
+	</xacro:d435_camera>
+	  <xacro:property name="camera_fov" value="3.0"/>
+	  <xacro:property name="camera_width" value="640"/>
+	  <xacro:property name="camera_height" value="480"/>
+	  <xacro:property name="camera_near" value="0.01"/>
+	  <xacro:property name="camera_far" value="100"/>
+	<xacro:d435_camera
+		parent="base_link"
+		name="z_base_camera"
+		camera_plugin="true">
+		<origin xyz="0.0 -0.3 -0.5" rpy="0.0  0.5 1.57"/>
 	</xacro:d435_camera>
 </xacro:if>
