Commit message: added bumper ee contact sensor (not publishing yet todo fix)

File: urdf/ur5.xacro (robot description, xacro)
@@ -63,4 +63,25 @@
       <selfCollide>true</selfCollide>
     </gazebo>
+	<!-- fix me https://answers.gazebosim.org//question/15095/gazebo-contact-sensor-added-to-a-robot-link-in-urdf-file-is-not-working-as-expected/-->
+	<!--gazebo reference="$(arg prefix)wrist_3_link">
+		<kp>1000000.0</kp>
+		<kd>100.0</kd>
+		<mu1>1.0</mu1>
+		<mu2>1.0</mu2>
+		<maxVel>1.0</maxVel>
+		<maxContacts>1</maxContacts>
+		<sensor name="ee_contact_sensor" type="contact">
+			<always_on>true</always_on>
+			<update_rate>250.0</update_rate>
+			<contact>
+				<collision>$(arg prefix)wrist_3_link_collision_collision</collision>
+			</contact>
+		        <plugin name="gazebo_ros_bumper_controller" filename="libgazebo_ros_bumper.so">
+				<bumperTopicName>/ur5/wrench</bumperTopicName>
+				<frameName>$(arg prefix)wrist_3_link</frameName>
+		        	<robotNamespace>ur5</robotNamespace>
+			</plugin>
+		</sensor>
+	</gazebo-->
     <!--
       Inject Gazebo ROS Control plugin, which allows us to use ros_control

Commit message: added realsense in simulation!
publishes in ee_camera topic

File: urdf/ur5.xacro (robot description, xacro)
@@ -2,4 +2,5 @@
 <robot xmlns:xacro="http://wiki.ros.org/xacro" name="ur_robot">
 <xacro:include filename="$(find ur_description)/urdf/inc/ur_macro.xacro"/>
+<xacro:arg name="vision_sensor" default="true"/>
 <xacro:arg name="gazebo" default="true"/>
 <xacro:arg name="prefix" default=""/>
@@ -27,4 +28,22 @@
 safety_pos_margin="$(arg safety_pos_margin)"
 safety_k_position="$(arg safety_k_position)"/>
+<xacro:if value="$(arg vision_sensor)">
+	<xacro:include filename="$(find ur_description)/sensors/d435_camera.urdf.xacro"/>
+	  <!-- realsense -->
+	  <!--These values are taken from  d435_camera.urdf.xacro and  d435_camera_openni.gazebo.urdf.xacro in sensors-description
+	 repo, commit 3fb6f787-->
+	  <xacro:property name="camera_fov" value="3.0"/>
+	  <xacro:property name="camera_width" value="640"/>
+	  <xacro:property name="camera_height" value="480"/>
+	  <xacro:property name="camera_near" value="0.1"/>
+	  <xacro:property name="camera_far" value="100"/>
+	  <xacro:property name="m_camera" value="0.07"/> <!--??-->
+	<xacro:d435_camera
+		parent="wrist_3_link"
+		name="ee_link"
+		camera_plugin="true">
+		<origin xyz="0.05 0.0 -0.02" rpy="0 -1.57 0.0"/>
+	</xacro:d435_camera>
+</xacro:if>
 <xacro:if value="$(arg gazebo)">
   <!--

Commit message: added gripper

File: urdf/ur5.xacro (robot description, xacro)
@@ -4,4 +4,5 @@
 <xacro:arg name="vision_sensor" default="true"/>
 <xacro:arg name="gazebo" default="true"/>
+<xacro:arg name="gripper" default="false"/>
 <xacro:arg name="prefix" default=""/>
 <xacro:arg name="transmission_hw_interface" default="hardware_interface/EffortJointInterface"/>
@@ -28,4 +29,12 @@
 safety_pos_margin="$(arg safety_pos_margin)"
 safety_k_position="$(arg safety_k_position)"/>
+<xacro:if value="$(arg gripper)">
+    <xacro:include filename="$(find gripper_description)/urdf/gripper.xacro"/>
+    <joint name="gripper_robot_joint" type="fixed">
+        <parent link="tool0"/>
+        <child link="gripper_base"/>
+        <origin xyz="0 0 0" rpy="0 0 0"/>
+    </joint>
+</xacro:if>
 <xacro:if value="$(arg vision_sensor)">
 	<xacro:include filename="$(find ur_description)/sensors/d435_camera.urdf.xacro"/>

Commit message: adjusted gripper orientation to be consistent with real robot

File: urdf/ur5.xacro (robot description, xacro)
@@ -36,5 +36,5 @@
         <parent link="tool0"/>
         <child link="gripper_base"/>
-        <origin xyz="0 0 0" rpy="0 0 0"/>
+        <origin xyz="0 0 0" rpy="0 0 3.14"/>
     </joint>
 </xacro:if>
