Commit message: adjusting go0 to avoid flickering

File: urdf/ur5.srdf.xacro (robot description, xacro)
@@ -4,5 +4,5 @@
     <joint name="shoulder_pan_joint" value="-0.32" />
     <joint name="shoulder_lift_joint" value="-0.78" />
-    <joint name="elbow_joint" value="-2.56" />
+    <joint name="elbow_joint" value="-2.1" />
     <joint name="wrist_1_joint" value="-1.63" />
     <joint name="wrist_2_joint" value="-1.57" />
