Commit message: added frames for potential fields algorithms

File: urdf/inc/ur_macro.xacro (robot description, xacro)
@@ -275,4 +275,23 @@
       <child link="${prefix}tool0"/>
     </joint>
+  <!-- fixed frames for collisions (potential fields)-->
+  <link name="upper_arm_link_middle"/>
+  <joint name="upper_arm_link_middle_fixed_joint" type="fixed">
+    <origin rpy="0 0 0" xyz="-${upperarm_inertia_length/2} 0 0.13"/>
+    <parent link="upper_arm_link"/>
+    <child link="upper_arm_link_middle"/>
+  </joint>
+  <link name="forearm_link_middle"/>
+  <joint name="forearm_link_middle_fixed_joint" type="fixed">
+    <origin rpy="0 0 0" xyz="${forearm_x/2} ${forearm_y/2} ${forearm_z/2}"/>
+    <parent link="forearm_link"/>
+    <child link="forearm_link_middle"/>
+  </joint>
+  <link name="forearm_link_end"/>
+  <joint name="forearm_link_end_fixed_joint" type="fixed">
+    <origin rpy="0 0 0" xyz="${forearm_x} ${forearm_y} ${forearm_z}"/>
+    <parent link="forearm_link"/>
+    <child link="forearm_link_end"/>
+  </joint>
   </xacro:macro>
 </robot>

Commit message: including properly gripper macro, IMPORTANT gripper is now always visible, and tool0 frame is in the middle of the hand,
if flag gripper is on then also trasmission are added to the joints
otherwise the gripper is a RIGID BODY

File: urdf/inc/ur_macro.xacro (robot description, xacro)
@@ -268,10 +268,10 @@
     </joint>
     <!-- ROS-Industrial 'tool0' frame: all-zeros tool frame -->
-    <link name="${prefix}tool0"/>
+    <link name="${prefix}tool0_without_gripper"/>
     <joint name="${prefix}flange-tool0" type="fixed">
       <!-- default toolframe: X+ left, Y+ up, Z+ front -->
       <origin xyz="0 0 0" rpy="${pi/2.0} 0 ${pi/2.0}"/>
       <parent link="${prefix}flange"/>
-      <child link="${prefix}tool0"/>
+      <child link="${prefix}tool0_without_gripper"/>
     </joint>
   <!-- fixed frames for collisions (potential fields)-->

File: urdf/ur5.urdf.xacro (robot description, xacro)
@@ -29,14 +29,15 @@
 safety_pos_margin="$(arg safety_pos_margin)"
 safety_k_position="$(arg safety_k_position)"/>
-<xacro:if value="$(arg gripper)">
-    <xacro:include filename="$(find gripper_description)/urdf/gripper.xacro">
- 		<xacro:arg name="transmission_hw_interface" value="$(arg transmission_hw_interface)"/>
-    </xacro:include>
-    <joint name="gripper_robot_joint" type="fixed">
-        <parent link="tool0"/>
+<xacro:include filename="$(find gripper_description)/urdf/gripper.macro.xacro" />
+<xacro:gripper
+	transmission_hw_interface="$(arg transmission_hw_interface)"
+	grasp_plugin="$(arg gripper)"
+	gripper_active="$(arg gripper)">
+</xacro:gripper>
+<joint name="gripper_robot_joint" type="fixed">
+        <parent link="tool0_without_gripper"/>
         <child link="gripper_base"/>
         <origin xyz="0 0 0" rpy="0 0 3.14"/>
-    </joint>
-</xacro:if>
+</joint>
 <xacro:if value="$(arg vision_sensor)">
 	<xacro:include filename="$(find ur_description)/sensors/d435_camera.urdf.xacro"/>
@@ -51,5 +52,5 @@
 	  <xacro:property name="m_camera" value="0.07"/> <!--??-->
 	<xacro:d435_camera
-		parent="tool0"
+		parent="wrist_3_link"
 		name="ee_camera"
 		camera_plugin="true">
